File: ecu_emu.sch (KiCad schematic (older format))
At the start: 29 parts, among them J1 Conn_01x04_Male, J2 Conn_02x06_Odd_Even, Q1 BCV46.215, U1 LD1117S33TR_SOT223, U2 TJA1021T, U3 STM32F105RBTx, Y1 Crystal KX-9A

Commit message: add README file, with svg graphics
Connections:
- wire segments 90 -> 122
Other:
- moved on the sheet: C1, C2, C3, C4, C5, C6, C7, D1, D2, D3, D4, J1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

Commit message: 1. solenoid rules with MOSFET and his driver 2. chane LIN to K-Bus cirquit 3. add shotky diod
Parts:
- removed C6: 4.7uF x 10V, Capacitors_SMD:C_1206, symbol CP
- removed C7: 1nF, Capacitors_SMD:C_0805, symbol C
- removed D1, D4: PMLL4148L.115, Diodes_SMD:D_SC-80, symbol D
- removed Q1: BCV46.215, TO_SOT_Packages_SMD:SOT-23, symbol Q_PNP_Darlington_BEC
- removed R10, R9: 1k, Resistors_SMD:R_0805, symbol R
- removed R11: 10k, Resistors_SMD:R_0805, symbol R
- removed U2: TJA1021T, Housings_SOIC:SOIC-8_3.9x4.9mm_Pitch1.27mm, symbol TJA1021T
- added C1: 10nF, Capacitors_SMD:C_0805, symbol C
- added C7, C8: 47uF x 16V, Capacitors_Tantalum_SMD:CP_Tantalum_Case-C_EIA-6032-28_Hand, symbol CP
- added C9: 1000 pF, Capacitors_SMD:C_0805, symbol C
- added D1: SS22A-SS210A-Galaxy, Diodes_SMD:D_SMA, symbol D_Schottky
- added Q1: IRF7201PBF, Housings_SOIC:SOIC-8_3.9x4.9mm_Pitch1.27mm, symbol IRF7201PBF
- added U3: FAN73711, Housings_SOIC:SOIC-8_3.9x4.9mm_Pitch1.27mm, symbol FAN73711
- added U4: E-L9637D, Housings_SOIC:SOIC-8_3.9x4.9mm_Pitch1.27mm, symbol E-L9637D
- D3: value PMLL4148L.115 -> SM4007; footprint Diodes_SMD:D_SC-80 -> Diodes_SMD:D_MELF_Handsoldering
- R8: value 1k5 -> 65
- U1: footprint TO_SOT_Packages_SMD:SOT-223-3Lead_TabPin2 -> TO_SOT_Packages_SMD:SOT-223-3_TabPin2
- renumbered C1 to C2, C2 to C4, C4 to C5, C5 to C6, J2 to J1, J1 to J2, U3 to U2
Connections:
- net labels added: +3V3, K-BUS_Vbatt, solenoid_driver, stm2K-BUS_UART_RX, stm2K-BUS_UART_TX
- net labels removed: LIN_Vbatt, stm2lin_SLEEP, stm2lin_UART_RX, stm2lin_UART_TX
- wire segments 122 -> 93
- no-connect marks 45 -> 50
Other:
- moved on the sheet: C2, C3, C6, D2, J1, U1

Commit message: sch: add resistor to hall sensor input
Parts:
- added R9: 1k, Resistors_SMD:R_0805, symbol R
- C2: footprint Capacitors_Tantalum_SMD:CP_Tantalum_Case-X_EIA-7343-43_Hand -> Capacitors_Tantalum_SMD:CP_Tantalum_Case-X_EIA-7343-43_Wave
- C7, C8: footprint Capacitors_Tantalum_SMD:CP_Tantalum_Case-C_EIA-6032-28_Hand -> Capacitors_Tantalum_SMD:CP_Tantalum_Case-C_EIA-6032-28_Wave
- D3: footprint Diodes_SMD:D_MELF_Handsoldering -> Diodes_SMD:D_MELF
Connections:
- net GND: now also R9.1
- net at R7.1, U2.11 (PC3/ADC1_IN13/ADC2_IN13): now also R9.2
